Commit message: Changes name of macro for inverted configuration

File: urs100_support/urdf/urs100_inverted_macro.xacro (robot description, xacro)
@@ -1,5 +1,5 @@
 <?xml version="1.0"?>
 <robot xmlns:xacro="http://wiki.ros.org/xacro">
-    <xacro:macro name="urs100" params="prefix parent *origin">
+    <xacro:macro name="urs100_inverted" params="prefix parent *origin">
         <xacro:arg name="rotary_stage" default="false"/>
         <link

Commit message: Added set velocity functionality

File: urs100_support/urdf/urs100_inverted_macro.xacro (robot description, xacro)
@@ -1,120 +1,120 @@
 <?xml version="1.0"?>
 <robot xmlns:xacro="http://wiki.ros.org/xacro">
-    <xacro:macro name="urs100_inverted" params="prefix parent *origin">
-        <xacro:arg name="rotary_stage" default="false"/>
-        <link
-                name="inner_rotation_platform">
-            <visual>
-                <origin
-                        xyz="0 0 0"
-                        rpy="0 0 0"/>
-                <geometry>
-                    <mesh
-                            filename="package://urs100_support/meshes/visual/inner_rotation_platform.stl"/>
-                </geometry>
-                <material
-                        name="">
-                    <color
-                            rgba="0.12156862745098 0.119607843137255 0.133333333333333 1"/>
-                </material>
-            </visual>
-            <collision>
-                <origin
-                        xyz="0 0 0"
-                        rpy="0 0 0"/>
-                <geometry>
-                    <mesh
-                            filename="package://urs100_support/meshes/collision/inner_rotation_platform.stl"/>
-                </geometry>
-            </collision>
-        </link>
-        <link
-                name="rotation_platform">
-            <visual>
-                <origin
-                        xyz="0 0 0"
-                        rpy="0 0 0"/>
-                <geometry>
-                    <mesh
-                            filename="package://urs100_support/meshes/visual/rotation_platform.stl"/>
-                </geometry>
-                <material
-                        name="">
-                    <color
-                            rgba="0.792156862745098 0.819607843137255 0.933333333333333 1"/>
-                </material>
-            </visual>
-            <collision>
-                <origin
-                        xyz="0 0 0"
-                        rpy="0 0 0"/>
-                <geometry>
-                    <mesh
-                            filename="package://urs100_support/meshes/collision/rotation_platform.stl"/>
-                </geometry>
-            </collision>
-        </link>
-        <link
-                name="rotation_base">
-            <visual>
-                <origin
-                        xyz="0 0 0"
-                        rpy="0 0 0"/>
-                <geometry>
-                    <mesh
-                            filename="package://urs100_support/meshes/visual/rotation_base.stl"/>
-                </geometry>
-                <material
-                        name="">
-                    <color
-                            rgba="0.12156862745098 0.119607843137255 0.133333333333333 1"/>
-                </material>
-            </visual>
-            <collision>
-                <origin
-                        xyz="0 0 0"
-                        rpy="0 0 0"/>
-                <geometry>
-                    <mesh
-                            filename="package://urs100_support/meshes/collision/rotation_base.stl"/>
-                </geometry>
-            </collision>
-        </link>
-        <joint
-                name="rotation_plate"
-                type="fixed">
-            <origin
-                    xyz="0.0 -0.03725 0.0"
-                    rpy="-1.5707963267949 -2.157041537713704e-31 -6.028485090085621e-17"/>
-            <parent
-                    link="inner_rotation_platform"/>
-            <child
-                    link="rotation_platform"/>
-        </joint>
-        <joint
-                name="joint_urs100"
-                type="revolute">
+<xacro:macro name="urs100_inverted" params="prefix parent *origin">
+    <xacro:arg name="rotary_stage" default="false"/>
+    <link
+            name="inner_rotation_platform">
+        <visual>
             <origin
                     xyz="0 0 0"
-                    rpy="0.0 -3.3863885623857104e-49 0.0"/>
-            <parent
-                    link="rotation_platform"/>
-            <child
-                    link="rotation_base"/>
-            <axis
-                    xyz="0 0 1"/>
-            <limit lower="${radians(-165.0)}" upper="${radians(165.0)}" effort="0.0" velocity="0.0"/>
-        </joint>
-        <joint
-                name="base_stage"
-                type="fixed">
+                    rpy="0 0 0"/>
+            <geometry>
+                <mesh
+                        filename="package://urs100_support/meshes/visual/inner_rotation_platform.stl"/>
+            </geometry>
+            <material
+                    name="">
+                <color
+                        rgba="0.12156862745098 0.119607843137255 0.133333333333333 1"/>
+            </material>
+        </visual>
+        <collision>
             <origin
-                    xyz="0.0 -1.08 -0.19"
-                    rpy="0.0 0.0 ${radians(90.0)}"/>
-            <parent
-                    link="rotation_base"/>
-            <child
-                    link="base_link"/>
-        </joint>
-    </xacro:macro>
+                    xyz="0 0 0"
+                    rpy="0 0 0"/>
+            <geometry>
+                <mesh
+                        filename="package://urs100_support/meshes/collision/inner_rotation_platform.stl"/>
+            </geometry>
+        </collision>
+    </link>
+    <link
+            name="rotation_platform">
+        <visual>
+            <origin
+                    xyz="0 0 0"
+                    rpy="0 0 0"/>
+            <geometry>
+                <mesh
+                        filename="package://urs100_support/meshes/visual/rotation_platform.stl"/>
+            </geometry>
+            <material
+                    name="">
+                <color
+                        rgba="0.792156862745098 0.819607843137255 0.933333333333333 1"/>
+            </material>
+        </visual>
+        <collision>
+            <origin
+                    xyz="0 0 0"
+                    rpy="0 0 0"/>
+            <geometry>
+                <mesh
+                        filename="package://urs100_support/meshes/collision/rotation_platform.stl"/>
+            </geometry>
+        </collision>
+    </link>
+    <link
+            name="rotation_base">
+        <visual>
+            <origin
+                    xyz="0 0 0"
+                    rpy="0 0 0"/>
+            <geometry>
+                <mesh
+                        filename="package://urs100_support/meshes/visual/rotation_base.stl"/>
+            </geometry>
+            <material
+                    name="">
+                <color
+                        rgba="0.12156862745098 0.119607843137255 0.133333333333333 1"/>
+            </material>
+        </visual>
+        <collision>
+            <origin
+                    xyz="0 0 0"
+                    rpy="0 0 0"/>
+            <geometry>
+                <mesh
+                        filename="package://urs100_support/meshes/collision/rotation_base.stl"/>
+            </geometry>
+        </collision>
+    </link>
+    <joint
+            name="rotation_plate"
+            type="fixed">
+        <origin
+                xyz="0.0 -0.03725 0.0"
+                rpy="-1.5707963267949 -2.157041537713704e-31 -6.028485090085621e-17"/>
+        <parent
+                link="inner_rotation_platform"/>
+        <child
+                link="rotation_platform"/>
+    </joint>
+    <joint
+            name="joint_urs100"
+            type="revolute">
+        <origin
+                xyz="0 0 0"
+                rpy="0.0 -3.3863885623857104e-49 0.0"/>
+        <parent
+                link="rotation_platform"/>
+        <child
+                link="rotation_base"/>
+        <axis
+                xyz="0 0 1"/>
+        <limit lower="${radians(-165.0)}" upper="${radians(165.0)}" effort="0.0" velocity="0.0"/>
+    </joint>
+    <joint
+            name="base_stage"
+            type="fixed">
+        <origin
+                xyz="0.0 -0.93 -0.205"
+                rpy="0.0 0.0 ${radians(90.0)}"/>
+        <parent
+                link="rotation_base"/>
+        <child
+                link="base_link"/>
+    </joint>
+</xacro:macro>
 </robot>

File: urs100_support/urdf/urs100_macro.xacro (robot description, xacro)
@@ -87,5 +87,5 @@
         </joint>
         <joint name="base_stage" type="fixed">
-            <origin rpy="0.0151101321324 -0.00591980854257 -1.57079632679" xyz="0.918991153433 -0.261224724446 0.199700111584" />
+            <origin rpy="-0.00603762215549 -0.00335447579975 -1.57079632679" xyz="0.919514000262 -0.261610857563 0.189064256822" />
             <parent link="${parent}" />
             <child link="rotation_base" />
